File: picostation_pcb.kicad_sch (KiCad schematic)
At the start: 17 parts, among them J1 Conn_01x06_Female, J2 Conn_01x20_Female, J3 PICO, J4 Conn_02x10_Female, J5 Conn_01x10_Socket, U1 LM78M05_TO252

Commit message: save
Parts:
- removed RN1: 10K, Resistor_THT:R_Array_SIP5, symbol Device:R_Network04
- added R2, R3, R4, R5: 10k, Resistor_SMD:R_0603_1608Metric_Pad0.98x0.95mm_HandSolder, symbol Device:R
- J1: footprint paulo:SD -> Connector_PinHeader_2.54mm:PinHeader_1x06_P2.54mm_Vertical
- J5: footprint (none) -> Connector_Card:microSD_HC_Hirose_DM3AT-SF-PEJM5
- renumbered C3 to C1, C1 to C3
Connections:
- net +3V3: now also R2.1, R3.1, R4.1, R5.1
- net pico_GP10: now also R4.2
- net pico_GP11: now also R3.2
- net pico_GP8: now also R5.2
- net at J5.10 (Pin_10), J5.3 (Pin_3): now also R2.2
Changed lines of the file:
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@@
   (junction (at 234.95 69.85) (diameter 0) (color 0 0 0 0)
   )
+  (junction (at 38.1 63.5) (diameter 0) (color 0 0 0 0)
+  )
   (junction (at 234.95 64.77) (diameter 0) (color 0 0 0 0)
   )
@@
   (junction (at 234.95 72.39) (diameter 0) (color 0 0 0 0)
   )
+  (junction (at 39.37 63.5) (diameter 0) (color 0 0 0 0)
+  )
   (junction (at 234.95 49.53) (diameter 0) (color 0 0 0 0)
   )
@@
   )
   (junction (at 27.94 26.67) (diameter 0) (color 0 0 0 0)
+  )
+  (junction (at 40.64 63.5) (diameter 0) (color 0 0 0 0)
   )
   (junction (at 234.95 36.83) (diameter 0) (color 0 0 0 0)
@@
     (stroke (width 0) (type default))
   )
+  (wire (pts (xy 39.37 60.96) (xy 39.37 63.5))
+    (stroke (width 0) (type default))
+  )
   (wire (pts (xy 38.1 71.12) (xy 38.1 90.17))
     (stroke (width 0) (type default))
@@
     (stroke (width 0) (type default))
   )
+  (wire (pts (xy 40.64 63.5) (xy 43.18 63.5))
+    (stroke (width 0) (type default))
+  )
   (wire (pts (xy 53.34 93.98) (xy 53.34 104.14))
     (stroke (width 0) (type default))
@@
     (stroke (width 0) (type default))
   )
+  (wire (pts (xy 39.37 63.5) (xy 40.64 63.5))
+    (stroke (width 0) (type default))
+  )
   (wire (pts (xy 210.82 24.13) (xy 234.95 24.13))
     (stroke (width 0) (type default))
@@
     (stroke (width 0) (type default))
   )
+  (wire (pts (xy 35.56 63.5) (xy 38.1 63.5))
+    (stroke (width 0) (type default))
+  )
   (wire (pts (xy 45.72 104.14) (xy 45.72 110.49))
     (stroke (width 0) (type default))
@@
   )
   (wire (pts (xy 24.13 26.67) (xy 27.94 26.67))
+    (stroke (width 0) (type default))
+  )
+  (wire (pts (xy 38.1 63.5) (xy 39.37 63.5))
     (stroke (width 0) (type default))
   )
@@
     )
   )
+  (symbol (lib_id "Device:R") (at 38.1 67.31 0) (unit 1)
+    (in_bom yes) (on_board yes) (dnp no) (fields_autoplaced)
+    (property "Reference" "R3" (at 40.64 66.675 0)
+      (effects (font (size 1.27 1.27)) (justify left))
+    )
+    (property "Value" "10k" (at 40.64 69.215 0)
+      (effects (font (size 1.27 1.27)) (justify left))
+    )
+    (property "Footprint" "Resistor_SMD:R_0603_1608Metric_Pad0.98x0.95mm_HandSolder" (at 36.322 67.31 90)
+      (effects (font (size 1.27 1.27)) hide)
+    )
+    (property "Datasheet" "~" (at 38.1 67.31 0)
+      (effects (font (size 1.27 1.27)) hide)
+    )
+    (pin "1")
+    (pin "2")
+    (instances
+      (project "picostation_pcb"
+        (path "/69032557-405f-457b-8a9a-4ca4fb07928c"
+          (reference "R3") (unit 1)
+        )
+      )
+    )
+  )
   (symbol (lib_id "power:+3V3") (at 165.1 113.03 0) (unit 1)
     (in_bom yes) (on_board yes) (dnp no) (fields_autoplaced)
@@
   (symbol (lib_id "Device:C") (at 49.53 104.14 90) (unit 1)
     (in_bom yes) (on_board yes) (dnp no) (fields_autoplaced)
-    (property "Reference" "C1" (at 49.53 97.79 90)
+    (property "Reference" "C3" (at 49.53 97.79 90)
       (effects (font (size 1.27 1.27)))
     )
@@
       (project "picostation_pcb"
         (path "/69032557-405f-457b-8a9a-4ca4fb07928c"
-          (reference "C1") (unit 1)
+          (reference "C3") (unit 1)
         )
       )
@@
     )
   )
+  (symbol (lib_id "Device:R") (at 35.56 67.31 0) (unit 1)
+    (in_bom yes) (on_board yes) (dnp no) (fields_autoplaced)
+    (property "Reference" "R2" (at 38.1 66.675 0)
+      (effects (font (size 1.27 1.27)) (justify left))
+    )
+    (property "Value" "10k" (at 38.1 69.215 0)
+      (effects (font (size 1.27 1.27)) (justify left))
+    )
+    (property "Footprint" "Resistor_SMD:R_0603_1608Metric_Pad0.98x0.95mm_HandSolder" (at 33.782 67.31 90)
+      (effects (font (size 1.27 1.27)) hide)
+    )
+    (property "Datasheet" "~" (at 35.56 67.31 0)
+      (effects (font (size 1.27 1.27)) hide)
+    )
+    (pin "1")
+    (pin "2")
+    (instances
+      (project "picostation_pcb"
+        (path "/69032557-405f-457b-8a9a-4ca4fb07928c"
+          (reference "R2") (unit 1)
+        )
+      )
+    )
+  )
   (symbol (lib_id "Mechanical:MountingHole_Pad") (at 83.82 20.32 0) (unit 1)
     (in_bom yes) (on_board yes) (dnp no) (fields_autoplaced)
@@
         (path "/69032557-405f-457b-8a9a-4ca4fb07928c"
           (reference "R1") (unit 1)
-        )
-      )
-    )
-  )
-  (symbol (lib_id "Device:R_Network04") (at 40.64 66.04 0) (unit 1)
-    (in_bom yes) (on_board yes) (dnp no) (fields_autoplaced)
-    (property "Reference" "RN1" (at 45.72 65.659 0)
-      (effects (font (size 1.27 1.27)) (justify left))
-    )
-    (property "Value" "10K" (at 45.72 68.199 0)
-      (effects (font (size 1.27 1.27)) (justify left))
-    )
-    (property "Footprint" "Resistor_THT:R_Array_SIP5" (at 47.625 66.04 90)
-      (effects (font (size 1.27 1.27)) hide)
-    )
-    (property "Datasheet" "http://www.vishay.com/docs/31509/csc.pdf" (at 40.64 66.04 0)
-      (effects (font (size 1.27 1.27)) hide)
-    )
-    (pin "1")
-    (pin "2")
-    (pin "3")
-    (pin "4")
-    (pin "5")
-    (instances
-      (project "picostation_pcb"
-        (path "/69032557-405f-457b-8a9a-4ca4fb07928c"
-          (reference "RN1") (unit 1)
         )
       )
@@
       (effects (font (size 1.27 1.27)))
     )
-    (property "Footprint" "" (at 25.4 90.17 0)
+    (property "Footprint" "Connector_Card:microSD_HC_Hirose_DM3AT-SF-PEJM5" (at 25.4 90.17 0)
       (effects (font (size 1.27 1.27)) hide)
     )
@@
   (symbol (lib_id "Device:C") (at 27.94 30.48 0) (unit 1)
     (in_bom yes) (on_board yes) (dnp no) (fields_autoplaced)
-    (property "Reference" "C3" (at 31.75 29.2099 0)
-      (effects (font (size 1.27 1.27)) (justify left))
-    )
-    (property "Value" "10u" (at 31.75 31.7499 0)
+    (property "Reference" "C1" (at 31.75 29.845 0)
+      (effects (font (size 1.27 1.27)) (justify left))
+    )
+    (property "Value" "10u" (at 31.75 32.385 0)
       (effects (font (size 1.27 1.27)) (justify left))
     )
@@
       (project "picostation_pcb"
         (path "/69032557-405f-457b-8a9a-4ca4fb07928c"
-          (reference "C3") (unit 1)
+          (reference "C1") (unit 1)
         )
       )
@@
         (path "/69032557-405f-457b-8a9a-4ca4fb07928c"
           (reference "H1") (unit 1)
+        )
+      )
+    )
+  )
+  (symbol (lib_id "Device:R") (at 40.64 67.31 0) (unit 1)
+    (in_bom yes) (on_board yes) (dnp no) (fields_autoplaced)
+    (property "Reference" "R4" (at 43.18 66.675 0)
+      (effects (font (size 1.27 1.27)) (justify left))
+    )
+    (property "Value" "10k" (at 43.18 69.215 0)
+      (effects (font (size 1.27 1.27)) (justify left))
+    )
+    (property "Footprint" "Resistor_SMD:R_0603_1608Metric_Pad0.98x0.95mm_HandSolder" (at 38.862 67.31 90)
+      (effects (font (size 1.27 1.27)) hide)
+    )
+    (property "Datasheet" "~" (at 40.64 67.31 0)
+      (effects (font (size 1.27 1.27)) hide)
+    )
+    (pin "1")
+    (pin "2")
+    (instances
+      (project "picostation_pcb"
+        (path "/69032557-405f-457b-8a9a-4ca4fb07928c"
+          (reference "R4") (unit 1)
+        )
+      )
+    )
+  )
+  (symbol (lib_id "Device:R") (at 43.18 67.31 0) (unit 1)
+    (in_bom yes) (on_board yes) (dnp no) (fields_autoplaced)
+    (property "Reference" "R5" (at 45.72 66.675 0)
+      (effects (font (size 1.27 1.27)) (justify left))
+    )
+    (property "Value" "10k" (at 45.72 69.215 0)
+      (effects (font (size 1.27 1.27)) (justify left))
+    )
+    (property "Footprint" "Resistor_SMD:R_0603_1608Metric_Pad0.98x0.95mm_HandSolder" (at 41.402 67.31 90)
+      (effects (font (size 1.27 1.27)) hide)
+    )
+    (property "Datasheet" "~" (at 43.18 67.31 0)
+      (effects (font (size 1.27 1.27)) hide)
+    )
+    (pin "1")
+    (pin "2")
+    (instances
+      (project "picostation_pcb"
+        (path "/69032557-405f-457b-8a9a-4ca4fb07928c"
+          (reference "R5") (unit 1)
         )
       )
@@
       (effects (font (size 1.27 1.27)))
     )
-    (property "Footprint" "paulo:SD" (at 66.04 88.9 0)
+    (property "Footprint" "Connector_PinHeader_2.54mm:PinHeader_1x06_P2.54mm_Vertical" (at 66.04 88.9 0)
       (effects (font (size 1.27 1.27)) hide)
     )
@@
     )
   )
-  (symbol (lib_id "power:+3V3") (at 35.56 60.96 0) (unit 1)
-    (in_bom yes) (on_board yes) (dnp no) (fields_autoplaced)
-    (property "Reference" "#PWR011" (at 35.56 64.77 0)
-      (effects (font (size 1.27 1.27)) hide)
-    )
-    (property "Value" "+3V3" (at 35.56 57.15 0)
-      (effects (font (size 1.27 1.27)))
-    )
-    (property "Footprint" "" (at 35.56 60.96 0)
-      (effects (font (size 1.27 1.27)) hide)
-    )
-    (property "Datasheet" "" (at 35.56 60.96 0)
-      (effects (font (size 1.27 1.27)) hide)
-    )
+  (symbol (lib_id "power:+3V3") (at 39.37 60.96 0) (unit 1)
+    (in_bom yes) (on_board yes) (dnp no) (fields_autoplaced)
+    (property "Reference" "#PWR011" (at 39.37 64.77 0)
+      (effects (font (size 1.27 1.27)) hide)
+    )
+    (property "Value" "+3V3" (at 39.37 57.15 0)
+      (effects (font (size 1.27 1.27)))
+    )
+    (property "Footprint" "" (at 39.37 60.96 0)
+      (effects (font (size 1.27 1.27)) hide)
+    )
+    (property "Datasheet" "" (at 39.37 60.96 0)
+      (effects (font (size 1.27 1.27)) hide)
+    )
